Commit message: feat: Removed packages for map creation that would not have contributed to the project. Added a launch file in the main package to launch the rtabmap_ros package

File: src/my_robot/urdf/my_robot.xacro (robot description, xacro)
@@ -185,3 +185,10 @@
 	<axis xyz="0 1 0"/>
 </joint>
+<joint name="camera_optical_joint" type="fixed">
+    <origin xyz="0 0 0" rpy="-1.5707 0 -1.5707"/>
+    <parent link="camera"/>
+    <child link="camera_link_optical"/>
+  </joint>
+<link name="camera_link_optical">
+</link>
 </robot>

Commit message: feat: Added localization file, modified mapping launch file to remap params

File: src/my_robot/urdf/my_robot.xacro (robot description, xacro)
@@ -160,4 +160,6 @@
 	<axis xyz="0 1 0" rpy="0 0 0"/>
 </joint>
+<link name="camera_link_optical">
+</link>
 <link name="hokuyo">
 	<visual name="hokuyo_visual">
@@ -190,5 +192,3 @@
     <child link="camera_link_optical"/>
   </joint>
-<link name="camera_link_optical">
-</link>
 </robot>
